File: KiCad/Mixer/Mixer.kicad_pcb (KiCad board)
At the start: 2 copper layers, 129.5 x 121.9 mm, 53 parts, among them J1 In 1.4, J10 In 2.4, J11 Mix Stereo Out, J2 In 1.3, J3 In 1.2, J4 In 1.1, J5 Out 1, J6 Out 2, J7 In 2.1, J8 In 2.2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

Commit message: Mixer PCB WIP
Parts:
- added REF**: M5mm_Pad_Via, MountingHole:MountingHole_5mm_Pad_Via, F.Cu at (91.4, 33.0)
- added REF**: M5mm_Pad_Via, MountingHole:MountingHole_5mm_Pad_Via, F.Cu at (91.4, 157.5)
- H5: moved to B.Cu
- J1, J10, J2, J3, J4, J5, J6, J7, J8, J9: footprint PCM_4ms_Jack:QuarterInch_Stereo_Vert_SwitchCraftNYS234-3 -> Connector_Audio:Jack_6.35mm_Neutrik_NJ2FD-V_Vertical
- J11: footprint PCM_4ms_Jack:QuarterInch_Stereo_Vert_2Switches_REAN-NYS232 -> Connector_Audio:Jack_6.35mm_Neutrik_NJ3FD-V_Vertical
- moved AMP2 135.7 mm to (111.0, 142.2)
- moved J6 108.0 mm to (125.1, 132.7)
- moved AMP1 104.8 mm to (97.2, 142.1)
- moved J5 103.3 mm to (109.2, 150.5)
- moved J11 98.7 mm to (125.1, 150.5)
- moved D1 37.0 mm to (50.8, 30.5)
- moved D2 37.0 mm to (50.8, 35.6)
- moved U1 22.9 mm to (69.9, 55.9)
- moved H5 20.7 mm to (54.6, 152.4), turned to 180 degrees
Other:
- board outline removed
