File: KiCad/Mixer/Mixer.kicad_sch (KiCad schematic)
At the start: 1 part, among them U1 TL072

Commit message: Mixer Schematic V1
Parts:
- removed U1: TL072, symbol Amplifier_Operational:TL072
- added AMP1, AMP2, MIX1.1, MIX1.2, MIX1.3, MIX1.4, MIX1.5, MIX1.6, MIX1.7, MIX1.8: 100k, symbol Device:R_Potentiometer
- added C1, C2, C5, C6: 47pF, Capacitor_THT:C_Disc_D3.0mm_W2.0mm_P2.50mm, symbol PCM_SL_Devices:Capacitor_NP
- added C3, C4: 100nF, Capacitor_THT:C_Disc_D3.0mm_W2.0mm_P2.50mm, symbol PCM_SL_Devices:Capacitor_NP
- added C7, C8: 10uF, symbol Device:C_Polarized_Small
- added D1, D2: 1N4001, Diode_THT:D_DO-41_SOD81_P10.16mm_Horizontal, symbol Diode:1N4001
- added J1: In 1.4, symbol Connector_Audio:AudioJack2
- added J10: In 2.4, symbol Connector_Audio:AudioJack2
- added J11: Mix Stereo Out, symbol Connector_Audio:AudioJack3
- added J2: In 1.3, symbol Connector_Audio:AudioJack2
- added J3: In 1.2, symbol Connector_Audio:AudioJack2
- added J4: In 1.1, symbol Connector_Audio:AudioJack2
- added J5: Out 1, symbol Connector_Audio:AudioJack2
- added J6: Out 2, symbol Connector_Audio:AudioJack2
- added J7: In 2.1, symbol Connector_Audio:AudioJack2
- added J8: In 2.2, symbol Connector_Audio:AudioJack2
- added J9: In 2.3, symbol Connector_Audio:AudioJack2
- added Q1, Q2: 2N3904, Package_TO_SOT_THT:TO-92_Inline, symbol Transistor_BJT:2N3904
- added R1, R10, R11, R12, R13, R14, R2, R5, R6, R7, R8, R9: 100k, Resistor_THT:R_Axial_DIN0207_L6.3mm_D2.5mm_P10.16mm_Horizontal, symbol PCM_SL_Devices:Resistor
- added R15, R16, R3, R4: 10k, Resistor_THT:R_Axial_DIN0207_L6.3mm_D2.5mm_P10.16mm_Horizontal, symbol PCM_SL_Devices:Resistor
- added SIGNAL1, SIGNAL2: LED, symbol Device:LED
- added U1: TL074, symbol Amplifier_Operational:TL074
Connections:
- new net: AMP2.1, C5.1, R10.2, R11.2, R12.2, R9.2, U1.9 (-)
- new net: AMP2.2, C5.2, R13.1, U1.8
- new net: C6.1, R13.2, R14.1, U1.13 (-)
- new net: C6.2, D2.2 (A), J11.R, J6.T, R14.2, U1.14
- new net: Q2.3 (C), R16.1
- new net: J2.T, MIX1.3.1
- new net: J3.T, MIX1.2.1
- new net: MIX1.2.2, R6.1
- new net: MIX1.7.2, R11.1
- new net: J1.T, MIX1.4.1
- new net: AMP1.1, C1.1, R5.2, R6.2, R7.2, R8.2, U1.2 (-)
- new net: AMP1.2, C1.2, R1.1, U1.1
- new net: Q2.1 (E), SIGNAL2.2 (A)
- new net: J9.T, MIX1.7.1
- new net: MIX1.3.2, R7.1
- new net: Q2.2 (B), R15.2
- new net: C2.2, D1.2 (A), J11.T, J5.T, R2.2, U1.7
- new net: MIX1.8.2, R12.1
- new net: MIX1.4.2, R8.1
- new net: J8.T, MIX1.6.1
- new net: C2.1, R1.2, R2.1, U1.6 (-)
- new net: MIX1.6.2, R10.1
- new net: Q1.3 (C), R4.1
- new net: J10.T, MIX1.8.1
- new net: D2.1 (K), R15.1
- new net: J4.T, MIX1.1.1
- new net: MIX1.1.2, R5.1
- new net: J7.T, MIX1.5.1
- new net: MIX1.5.2, R9.1
- new net: Q1.1 (E), SIGNAL1.2 (A)
- new net: Q1.2 (B), R3.2
- new net: D1.1 (K), R3.1
- new net +10: C3.2, C7.1, U1.4 (V+)
- new net +5V: R16.2, R4.2
- new net -12: C4.2, C8.2, U1.11 (V-)
- new net GND: C3.1, C4.1, C7.2, C8.1, J1.S, J10.S, J11.S, J2.S, J3.S, J4.S, J5.S, J6.S, J7.S, J8.S, J9.S, MIX1.1.3, MIX1.2.3, MIX1.3.3, MIX1.4.3, MIX1.5.3, MIX1.6.3, MIX1.7.3, MIX1.8.3, SIGNAL1.1 (K), SIGNAL2.1 (K), U1.10 (+), U1.12 (+), U1.3 (+), U1.5 (+)
- no-connect marks 0 -> 2
Other:
- note added: "CV/DC coupled!"
- note added: "Check poles on pots so rotation is correct direction"
- note added: "Decoupling caps"
- note added: "Mixed Stereo Out (hot!)"
- note added: "Mixer 1"
- note added: "Mixer 2"
- note added: "T = Left R = Right S = Ground"
- note removed: "100nf & 10uf decoupling caps on op amp power!"
- note removed: "4 inputs 1 output x2"
- note removed: "Audio/AC coupled"
- note removed: "CV/DC coupled"

Commit message: Arranged mixer footprints
Parts:
- AMP1, AMP2, MIX1.1, MIX1.2, MIX1.3, MIX1.4: footprint (none) -> PCM_4ms_Potentiometer:Pot_9mm_DShaft
- C7, C8: footprint (none) -> PCM_4ms_Capacitor:CP_Radial_P2.5mm
- J1, J10, J2, J3, J4, J5, J6, J7, J8, J9: footprint (none) -> PCM_4ms_Jack:QuarterInch_Stereo_Vert_SwitchCraftNYS234-3
- J11: footprint (none) -> PCM_4ms_Jack:QuarterInch_Stereo_Vert_2Switches_REAN-NYS232
- MIX2.1: renamed from MIX1.5; footprint (none) -> PCM_4ms_Potentiometer:Pot_9mm_DShaft
- MIX2.2: renamed from MIX1.6; footprint (none) -> PCM_4ms_Potentiometer:Pot_9mm_DShaft
- MIX2.3: renamed from MIX1.7; footprint (none) -> PCM_4ms_Potentiometer:Pot_9mm_DShaft
- MIX2.4: renamed from MIX1.8; footprint (none) -> PCM_4ms_Potentiometer:Pot_9mm_DShaft
- SIGNAL1, SIGNAL2: footprint (none) -> PCM_4ms_LED:LED_3mm_C1A2_Polarity_Indicator
- U1: footprint (none) -> PCM_4ms_Package_DIP:DIP-14_W7.62mm
Changed lines of the file:
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@@
       (effects (font (size 1.27 1.27)))
     )
-    (property "Footprint" "" (at 267.97 130.81 0)
+    (property "Footprint" "PCM_4ms_Capacitor:CP_Radial_P2.5mm" (at 267.97 130.81 0)
       (effects (font (size 1.27 1.27)) hide)
     )
@@
       (effects (font (size 1.27 1.27)) (justify right))
     )
-    (property "Footprint" "" (at 34.29 63.5 0)
+    (property "Footprint" "PCM_4ms_Jack:QuarterInch_Stereo_Vert_SwitchCraftNYS234-3" (at 34.29 63.5 0)
       (effects (font (size 1.27 1.27)) hide)
     )
@@
       (effects (font (size 1.27 1.27)) (justify right))
     )
-    (property "Footprint" "" (at 83.82 152.4 0)
+    (property "Footprint" "PCM_4ms_Potentiometer:Pot_9mm_DShaft" (at 83.82 152.4 0)
       (effects (font (size 1.27 1.27)) hide)
     )
@@
       (effects (font (size 1.27 1.27)))
     )
-    (property "Footprint" "" (at 123.19 128.27 0)
+    (property "Footprint" "PCM_4ms_Package_DIP:DIP-14_W7.62mm" (at 123.19 128.27 0)
       (effects (font (size 1.27 1.27)) hide)
     )
@@
       (effects (font (size 1.27 1.27)) (justify right))
     )
-    (property "Footprint" "" (at 50.8 50.8 0)
+    (property "Footprint" "PCM_4ms_Potentiometer:Pot_9mm_DShaft" (at 50.8 50.8 0)
       (effects (font (size 1.27 1.27)) hide)
     )
@@
       (effects (font (size 1.27 1.27)) (justify right))
     )
-    (property "Footprint" "" (at 34.29 80.01 0)
+    (property "Footprint" "PCM_4ms_Jack:QuarterInch_Stereo_Vert_SwitchCraftNYS234-3" (at 34.29 80.01 0)
       (effects (font (size 1.27 1.27)) hide)
     )
@@
       (effects (font (size 1.27 1.27)) (justify right))
     )
-    (property "Footprint" "" (at 154.94 130.81 0)
+    (property "Footprint" "PCM_4ms_LED:LED_3mm_C1A2_Polarity_Indicator" (at 154.94 130.81 0)
       (effects (font (size 1.27 1.27)) hide)
     )
@@
       (effects (font (size 1.27 1.27)) (justify right))
     )
-    (property "Footprint" "" (at 34.29 146.05 0)
+    (property "Footprint" "PCM_4ms_Jack:QuarterInch_Stereo_Vert_SwitchCraftNYS234-3" (at 34.29 146.05 0)
       (effects (font (size 1.27 1.27)) hide)
     )
@@
       (effects (font (size 1.27 1.27)) (justify right))
     )
-    (property "Footprint" "" (at 50.8 67.31 0)
+    (property "Footprint" "PCM_4ms_Potentiometer:Pot_9mm_DShaft" (at 50.8 67.31 0)
       (effects (font (size 1.27 1.27)) hide)
     )
@@
       (effects (font (size 1.27 1.27)))
     )
-    (property "Footprint" "" (at 223.52 91.44 0)
+    (property "Footprint" "PCM_4ms_Jack:QuarterInch_Stereo_Vert_2Switches_REAN-NYS232" (at 223.52 91.44 0)
       (effects (font (size 1.27 1.27)) hide)
     )
@@
       (effects (font (size 1.27 1.27)) (justify right))
     )
-    (property "Footprint" "" (at 34.29 129.54 0)
+    (property "Footprint" "PCM_4ms_Jack:QuarterInch_Stereo_Vert_SwitchCraftNYS234-3" (at 34.29 129.54 0)
       (effects (font (size 1.27 1.27)) hide)
     )
@@
       (effects (font (size 1.27 1.27)))
     )
-    (property "Footprint" "" (at 90.17 48.26 0)
+    (property "Footprint" "PCM_4ms_Package_DIP:DIP-14_W7.62mm" (at 90.17 48.26 0)
       (effects (font (size 1.27 1.27)) hide)
     )
@@
       (effects (font (size 1.27 1.27)) (justify right))
     )
-    (property "Footprint" "" (at 34.29 46.99 0)
+    (property "Footprint" "PCM_4ms_Jack:QuarterInch_Stereo_Vert_SwitchCraftNYS234-3" (at 34.29 46.99 0)
       (effects (font (size 1.27 1.27)) hide)
     )
@@
   (symbol (lib_id "Device:R_Potentiometer") (at 50.8 133.35 0) (unit 1)
     (in_bom yes) (on_board yes) (dnp no)
-    (property "Reference" "MIX1.6" (at 49.53 132.08 0)
+    (property "Reference" "MIX2.2" (at 49.53 132.08 0)
       (effects (font (size 1.27 1.27)) (justify right))
     )
@@
       (effects (font (size 1.27 1.27)) (justify right))
     )
-    (property "Footprint" "" (at 50.8 133.35 0)
+    (property "Footprint" "PCM_4ms_Potentiometer:Pot_9mm_DShaft" (at 50.8 133.35 0)
       (effects (font (size 1.27 1.27)) hide)
     )
@@
       (project "Mixer"
         (path "/7953a940-4dd3-4ecd-9e3a-aee4f61292de"
-          (reference "MIX1.6") (unit 1)
+          (reference "MIX2.2") (unit 1)
         )
       )
@@
   (symbol (lib_id "Device:R_Potentiometer") (at 50.8 166.37 0) (unit 1)
     (in_bom yes) (on_board yes) (dnp no)
-    (property "Reference" "MIX1.8" (at 49.53 165.1 0)
+    (property "Reference" "MIX2.4" (at 49.53 165.1 0)
       (effects (font (size 1.27 1.27)) (justify right))
     )
@@
       (effects (font (size 1.27 1.27)) (justify right))
     )
-    (property "Footprint" "" (at 50.8 166.37 0)
+    (property "Footprint" "PCM_4ms_Potentiometer:Pot_9mm_DShaft" (at 50.8 166.37 0)
       (effects (font (size 1.27 1.27)) hide)
     )
@@
       (project "Mixer"
         (path "/7953a940-4dd3-4ecd-9e3a-aee4f61292de"
-          (reference "MIX1.8") (unit 1)
+          (reference "MIX2.4") (unit 1)
         )
       )
@@
   (symbol (lib_id "Device:R_Potentiometer") (at 50.8 149.86 0) (unit 1)
     (in_bom yes) (on_board yes) (dnp no)
-    (property "Reference" "MIX1.7" (at 49.53 148.59 0)
+    (property "Reference" "MIX2.3" (at 49.53 148.59 0)
       (effects (font (size 1.27 1.27)) (justify right))
     )
@@
       (effects (font (size 1.27 1.27)) (justify right))
     )
-    (property "Footprint" "" (at 50.8 149.86 0)
+    (property "Footprint" "PCM_4ms_Potentiometer:Pot_9mm_DShaft" (at 50.8 149.86 0)
       (effects (font (size 1.27 1.27)) hide)
     )
@@
       (project "Mixer"
         (path "/7953a940-4dd3-4ecd-9e3a-aee4f61292de"
-          (reference "MIX1.7") (unit 1)
+          (reference "MIX2.3") (unit 1)
         )
       )
@@
       (effects (font (size 1.27 1.27)))
     )
-    (property "Footprint" "" (at 170.18 152.4 0)
+    (property "Footprint" "PCM_4ms_Jack:QuarterInch_Stereo_Vert_SwitchCraftNYS234-3" (at 170.18 152.4 0)
       (effects (font (size 1.27 1.27)) hide)
     )
@@
       (effects (font (size 1.27 1.27)) (justify right))
     )
-    (property "Footprint" "" (at 50.8 34.29 0)
+    (property "Footprint" "PCM_4ms_Potentiometer:Pot_9mm_DShaft" (at 50.8 34.29 0)
       (effects (font (size 1.27 1.27)) hide)
     )
@@
       (effects (font (size 1.27 1.27)) (justify right))
     )
-    (property "Footprint" "" (at 34.29 113.03 0)
+    (property "Footprint" "PCM_4ms_Jack:QuarterInch_Stereo_Vert_SwitchCraftNYS234-3" (at 34.29 113.03 0)
       (effects (font (size 1.27 1.27)) hide)
     )
@@
       (effects (font (size 1.27 1.27)) (justify right))
     )
-    (property "Footprint" "" (at 50.8 83.82 0)
+    (property "Footprint" "PCM_4ms_Potentiometer:Pot_9mm_DShaft" (at 50.8 83.82 0)
       (effects (font (size 1.27 1.27)) hide)
     )
@@
   (symbol (lib_id "Device:R_Potentiometer") (at 50.8 116.84 0) (unit 1)
     (in_bom yes) (on_board yes) (dnp no)
-    (property "Reference" "MIX1.5" (at 49.53 115.57 0)
+    (property "Reference" "MIX2.1" (at 49.53 115.57 0)
       (effects (font (size 1.27 1.27)) (justify right))
     )
@@
       (effects (font (size 1.27 1.27)) (justify right))
     )
-    (property "Footprint" "" (at 50.8 116.84 0)
+    (property "Footprint" "PCM_4ms_Potentiometer:Pot_9mm_DShaft" (at 50.8 116.84 0)
       (effects (font (size 1.27 1.27)) hide)
     )
@@
       (project "Mixer"
         (path "/7953a940-4dd3-4ecd-9e3a-aee4f61292de"
-          (reference "MIX1.5") (unit 1)
+          (reference "MIX2.1") (unit 1)
         )
       )
@@
       (effects (font (size 1.27 1.27)) (justify right))
     )
-    (property "Footprint" "" (at 34.29 30.48 0)
+    (property "Footprint" "PCM_4ms_Jack:QuarterInch_Stereo_Vert_SwitchCraftNYS234-3" (at 34.29 30.48 0)
       (effects (font (size 1.27 1.27)) hide)
     )
@@
       (effects (font (size 1.27 1.27)))
     )
-    (property "Footprint" "" (at 123.19 45.72 0)
+    (property "Footprint" "PCM_4ms_Package_DIP:DIP-14_W7.62mm" (at 123.19 45.72 0)
       (effects (font (size 1.27 1.27)) hide)
     )
@@
       (effects (font (size 1.27 1.27)))
     )
-    (property "Footprint" "" (at 267.97 153.67 0)
+    (property "Footprint" "PCM_4ms_Capacitor:CP_Radial_P2.5mm" (at 267.97 153.67 0)
       (effects (font (size 1.27 1.27)) hide)
     )
@@
       (effects (font (size 1.27 1.27)))
     )
-    (property "Footprint" "" (at 90.17 130.81 0)
+    (property "Footprint" "PCM_4ms_Package_DIP:DIP-14_W7.62mm" (at 90.17 130.81 0)
       (effects (font (size 1.27 1.27)) hide)
     )
@@
       (effects (font (size 1.27 1.27)) (justify right))
     )
-    (property "Footprint" "" (at 154.94 48.26 0)
+    (property "Footprint" "PCM_4ms_LED:LED_3mm_C1A2_Polarity_Indicator" (at 154.94 48.26 0)
       (effects (font (size 1.27 1.27)) hide)
     )
@@
       (effects (font (size 1.27 1.27)) (justify right))
     )
-    (property "Footprint" "" (at 83.82 69.85 0)
+    (property "Footprint" "PCM_4ms_Potentiometer:Pot_9mm_DShaft" (at 83.82 69.85 0)
       (effects (font (size 1.27 1.27)) hide)
     )
@@
       (effects (font (size 1.27 1.27)) (justify right))
     )
-    (property "Footprint" "" (at 34.29 162.56 0)
+    (property "Footprint" "PCM_4ms_Jack:QuarterInch_Stereo_Vert_SwitchCraftNYS234-3" (at 34.29 162.56 0)
       (effects (font (size 1.27 1.27)) hide)
     )
@@
       (effects (font (size 1.27 1.27)) (justify left))
     )
-    (property "Footprint" "" (at 260.35 139.7 0)
+    (property "Footprint" "PCM_4ms_Package_DIP:DIP-14_W7.62mm" (at 260.35 139.7 0)
       (effects (font (size 1.27 1.27)) hide)
     )
@@
       (effects (font (size 1.27 1.27)))
     )
-    (property "Footprint" "" (at 170.18 69.85 0)
-      (effects (font (size 1.27 1.27)) hide)
-    )
+    (property "Footprint" "PCM_4ms_Jack:QuarterInch_Stereo_Vert_SwitchCraftNYS234-3" (at 170.18 69.85 0)
+      (effects (font (size 1.27 1.27)) hide)
+    )

Commit message: Mixer PCB WIP
Parts:
- J1, J10, J2, J3, J4, J5, J6, J7, J8, J9: footprint PCM_4ms_Jack:QuarterInch_Stereo_Vert_SwitchCraftNYS234-3 -> Connector_Audio:Jack_6.35mm_Neutrik_NJ2FD-V_Vertical
- J11: footprint PCM_4ms_Jack:QuarterInch_Stereo_Vert_2Switches_REAN-NYS232 -> Connector_Audio:Jack_6.35mm_Neutrik_NJ3FD-V_Vertical
Changed lines of the file:
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@@
       (effects (font (size 1.27 1.27)) (justify right))
     )
-    (property "Footprint" "PCM_4ms_Jack:QuarterInch_Stereo_Vert_SwitchCraftNYS234-3" (at 34.29 63.5 0)
+    (property "Footprint" "Connector_Audio:Jack_6.35mm_Neutrik_NJ2FD-V_Vertical" (at 34.29 63.5 0)
       (effects (font (size 1.27 1.27)) hide)
     )
@@
       (effects (font (size 1.27 1.27)) (justify right))
     )
-    (property "Footprint" "PCM_4ms_Jack:QuarterInch_Stereo_Vert_SwitchCraftNYS234-3" (at 34.29 80.01 0)
+    (property "Footprint" "Connector_Audio:Jack_6.35mm_Neutrik_NJ2FD-V_Vertical" (at 34.29 80.01 0)
       (effects (font (size 1.27 1.27)) hide)
     )
@@
       (effects (font (size 1.27 1.27)) (justify right))
     )
-    (property "Footprint" "PCM_4ms_Jack:QuarterInch_Stereo_Vert_SwitchCraftNYS234-3" (at 34.29 146.05 0)
+    (property "Footprint" "Connector_Audio:Jack_6.35mm_Neutrik_NJ2FD-V_Vertical" (at 34.29 146.05 0)
       (effects (font (size 1.27 1.27)) hide)
     )
@@
       (effects (font (size 1.27 1.27)))
     )
-    (property "Footprint" "PCM_4ms_Jack:QuarterInch_Stereo_Vert_2Switches_REAN-NYS232" (at 223.52 91.44 0)
+    (property "Footprint" "Connector_Audio:Jack_6.35mm_Neutrik_NJ3FD-V_Vertical" (at 223.52 91.44 0)
       (effects (font (size 1.27 1.27)) hide)
     )
@@
       (effects (font (size 1.27 1.27)) (justify right))
     )
-    (property "Footprint" "PCM_4ms_Jack:QuarterInch_Stereo_Vert_SwitchCraftNYS234-3" (at 34.29 129.54 0)
+    (property "Footprint" "Connector_Audio:Jack_6.35mm_Neutrik_NJ2FD-V_Vertical" (at 34.29 129.54 0)
       (effects (font (size 1.27 1.27)) hide)
     )
@@
       (effects (font (size 1.27 1.27)) (justify right))
     )
-    (property "Footprint" "PCM_4ms_Jack:QuarterInch_Stereo_Vert_SwitchCraftNYS234-3" (at 34.29 46.99 0)
+    (property "Footprint" "Connector_Audio:Jack_6.35mm_Neutrik_NJ2FD-V_Vertical" (at 34.29 46.99 0)
       (effects (font (size 1.27 1.27)) hide)
     )
@@
       (effects (font (size 1.27 1.27)))
     )
-    (property "Footprint" "PCM_4ms_Jack:QuarterInch_Stereo_Vert_SwitchCraftNYS234-3" (at 170.18 152.4 0)
+    (property "Footprint" "Connector_Audio:Jack_6.35mm_Neutrik_NJ2FD-V_Vertical" (at 170.18 152.4 0)
       (effects (font (size 1.27 1.27)) hide)
     )
@@
       (effects (font (size 1.27 1.27)) (justify right))
     )
-    (property "Footprint" "PCM_4ms_Jack:QuarterInch_Stereo_Vert_SwitchCraftNYS234-3" (at 34.29 113.03 0)
+    (property "Footprint" "Connector_Audio:Jack_6.35mm_Neutrik_NJ2FD-V_Vertical" (at 34.29 113.03 0)
       (effects (font (size 1.27 1.27)) hide)
     )
@@
       (effects (font (size 1.27 1.27)) (justify right))
     )
-    (property "Footprint" "PCM_4ms_Jack:QuarterInch_Stereo_Vert_SwitchCraftNYS234-3" (at 34.29 30.48 0)
+    (property "Footprint" "Connector_Audio:Jack_6.35mm_Neutrik_NJ2FD-V_Vertical" (at 34.29 30.48 0)
       (effects (font (size 1.27 1.27)) hide)
     )
@@
       (effects (font (size 1.27 1.27)) (justify right))
     )
-    (property "Footprint" "PCM_4ms_Jack:QuarterInch_Stereo_Vert_SwitchCraftNYS234-3" (at 34.29 162.56 0)
+    (property "Footprint" "Connector_Audio:Jack_6.35mm_Neutrik_NJ2FD-V_Vertical" (at 34.29 162.56 0)
       (effects (font (size 1.27 1.27)) hide)
     )
@@
       (effects (font (size 1.27 1.27)))
     )
-    (property "Footprint" "PCM_4ms_Jack:QuarterInch_Stereo_Vert_SwitchCraftNYS234-3" (at 170.18 69.85 0)
-      (effects (font (size 1.27 1.27)) hide)
-    )
+    (property "Footprint" "Connector_Audio:Jack_6.35mm_Neutrik_NJ2FD-V_Vertical" (at 170.18 69.85 0)
+      (effects (font (size 1.27 1.27)) hide)
+    )
